File: kicad/byte.kicad_pcb (KiCad board)
At the start: 2 copper layers, 91.4 x 66 mm, 38 parts, among them J1 Barrel_Jack, SW1 RotaryEncoder_Switch, U1 ATtiny85-20P, U3 MAX6951

Commit message: revB
Parts:
- added R6: 10k, Resistor_SMD:R_1206_3216Metric_Pad1.30x1.75mm_HandSolder, F.Cu at (137.2, 95.2)
- R5: value 4k7 -> 1k
Connections:
- SW1 pad S2: GND -> Net-(R6-Pad1)
- U1 pad 1: unconnected-(U1-~{RESET}/PB5-Pad1) -> SWITCH
- U1 pad 6: SWITCH -> CS
- U3 pad 15: GND -> CS
Routing:
- net CS: track 0.00 -> 24.9 mm
- net Net-(R6-Pad1): track 0.00 -> 8.40 mm
- net SWITCH: track 51.8 -> 44.4 mm
- net GND: track 7.09 -> 2.36 mm
Other:
- board text added: "REVISION B JUNE 2023"
- board text removed: "REVISION A MARCH 2023"

Commit message: revC
Other:
- board text added: "REVISION C DECEMBER 2024"
- board text removed: "REVISION B JUNE 2023"
Changed lines of the file:
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@@
   (title_block
     (title "Byte Board")
-    (date "2023-06-05")
-    (rev "B")
+    (date "2024-01-16")
+    (rev "C")
     (company "University of Wisconsin-Madison")
     (comment 1 "Department of Chemistry")
@@
     (property "ki_keywords" "R res resistor")
     (attr smd)
-    (fp_text reference "R2" (at 0 -1.82) (layer "F.SilkS")
+    (fp_text reference "R2" (at 3.455 0) (layer "F.SilkS")
         (effects (font (size 1 1) (thickness 0.15)))
     )
-    (fp_text value "4k7" (at 0 1.82) (layer "F.Fab")
+    (fp_text value "4k7" (at -3.784 0) (layer "F.SilkS")
         (effects (font (size 1 1) (thickness 0.15)))
     )
@@
     (property "ki_keywords" "R res resistor")
     (attr smd)
-    (fp_text reference "R4" (at 0 -1.82) (layer "F.SilkS")
+    (fp_text reference "R4" (at 3.455 0) (layer "F.SilkS")
         (effects (font (size 1 1) (thickness 0.15)))
     )
-    (fp_text value "4k7" (at 0 1.82) (layer "F.Fab")
+    (fp_text value "4k7" (at -3.784 0) (layer "F.SilkS")
         (effects (font (size 1 1) (thickness 0.15)))
     )
@@
         (effects (font (size 1 1) (thickness 0.15)))
     )
-    (fp_text value "1k" (at 0 1.82) (layer "F.Fab")
+    (fp_text value "1k" (at 0 1.82) (layer "F.SilkS")
         (effects (font (size 1 1) (thickness 0.15)))
     )
@@
     (property "Sheetname" "")
     (attr through_hole)
-    (fp_text reference "PS1" (at -3.325 -9.135) (layer "F.SilkS")
+    (fp_text reference "PS1" (at -3.325 -9.135) (layer "F.Fab")
         (effects (font (size 1 1) (thickness 0.015)))
     )
@@
     (property "ki_keywords" "R res resistor")
     (attr smd)
-    (fp_text reference "R1" (at 0 -1.82) (layer "F.SilkS")
+    (fp_text reference "R1" (at -3.51 -0.1) (layer "F.SilkS")
         (effects (font (size 1 1) (thickness 0.15)))
     )
-    (fp_text value "1k" (at 0 1.82) (layer "F.Fab")
+    (fp_text value "1k" (at 3.49 -0.1) (layer "F.SilkS")
         (effects (font (size 1 1) (thickness 0.15)))
     )
@@
         (effects (font (size 1 1) (thickness 0.15)))
     )
-    (fp_text value "10k" (at 0 1.82) (layer "F.Fab")
+    (fp_text value "10k" (at 0 1.82) (layer "F.SilkS")
         (effects (font (size 1 1) (thickness 0.15)))
     )
@@
     (property "ki_keywords" "LED diode")
     (attr smd)
-    (fp_text reference "D9" (at 0 -1.82) (layer "F.SilkS")
+    (fp_text reference "D9" (at -0.01 -1.82) (layer "F.SilkS")
         (effects (font (size 1 1) (thickness 0.15)))
     )
@@
     (effects (font (size 1 1) (thickness 0.15)) (justify mirror))
   )
-  (gr_text "REVISION B\nJUNE 2023" (at 72.39 93.98 270) (layer "B.SilkS")
+  (gr_text "REVISION C\nDECEMBER 2024" (at 72.39 93.98 270) (layer "B.SilkS")
     (effects (font (size 1 1) (thickness 0.15)) (justify mirror))
   )
