File: kicad/byte.kicad_sch (KiCad schematic)
At the start: 14 parts, among them J1 Barrel_Jack, SW1 RotaryEncoder_Switch, U1 ATtiny85-20P

Commit message: revB
Parts:
- added R6: 10k, Resistor_SMD:R_1206_3216Metric_Pad1.30x1.75mm_HandSolder, symbol Device:R_US
- R5: value 4k7 -> 1k
Connections:
- net GND: now also R6.2; no longer SW1.S2
- net SWITCH: now also U1.1 (~{RESET}/PB5); no longer U1.6 (PB1)
- new net: R6.1, SW1.S2
- new net CS: U1.6 (PB1)
- no-connect marks 2 -> 1
Other:
- note added: "FORCED TO USE THE RESET PIN AS I/O YOU CAN DISABLE THE RESET PIN USING A FUSE, BUT THAT REQUIRES A SPECIAL PROGRAMMER THIS WILL WORK AS AN ANALOG INPUT, AS LONG AS IT REMAINS "HIGH ENOUGH" WILL NOT INTERRUPT TO RESET"
- note removed: "https://thewanderingengineer.com/2014/08/11/rotary-encoder-on-the-attiny85-part-2/"
- moved on the sheet: R5
